Commit message: ✅ Complete robot system with ball chaser
🎯 New Features:
- Added my_robot_bringup package: single launch file for entire system
- Added my_robot_chaser package: red ball tracking with camera
- JointStatePublisher plugin for proper /joint_states publishing
- RosClockPublisher in world file to prevent time jumps

🔧 Bug Fixes:
- Fixed /joint_states conflict (removed joint_state_publisher_gui)
- Fixed angular velocity signs in ball_chaser (left/right rotation)
- Added /joint_states bridge to ros_gz_bridge
- Fixed transform tree (world→odom→base_link→wheels/camera)

📦 System Components:
- Gazebo simulation with differential drive robot
- Camera sensor with HSV-based red ball detection
- Complete TF tree with static and dynamic transforms
- RViz visualization with camera feed
- Automated TF frames PDF generation

🚀 Launch:
ros2 launch my_robot_bringup bringup.launch.py

All systems operational! Robot successfully tracks red ball! 🔴🤖

File: src/my_robot_description/urdf/my_robot.urdf (robot description, URDF)
Before this commit: robot my_diff_drive_robot, 5 links, 4 joints
Joints:
- joint left_wheel_joint: limit (none) -> effort=1.0 velocity=1.0
- joint right_wheel_joint: limit (none) -> effort=1.0 velocity=1.0
